File: pcb/mcu_integration.kicad_pcb (KiCad board)
At the start: 4 copper layers, 70 x 70 mm, 77 parts, among them IC1 TL7660IDGKR, IC2 TL081IDT, IC3 LMT87DCKT, IC6 AD844_OPAMP_AL, IC7 FOD814_OPTO_AL, J1 Conn_01x05, J2 Conn_01x03, J5 DM3BT-DSF-PEJS, U1 STM32F103RBTx, U2 LTC4300A-1IMS8_PBF, U3 REF192_AL

Commit message: Added 3V3 linear voltage regulator
Parts:
- added C25: 2.2u, Capacitor_SMD:C_0402_1005Metric, F.Cu at (158.7, 75.2)
- added C26: 0.01u, Capacitor_SMD:C_0402_1005Metric, F.Cu at (155.7, 75.2)
- added C50: 0.1u, Capacitor_SMD:C_0402_1005Metric, F.Cu at (160.2, 70.7)
- added U4: TPS79933QDDCRQ1, TPS79933QDDCRQ1 (1):SOT95P280X110-5N, F.Cu at (157.2, 72.2)
- moved G*** 38.4 mm to (118.7, 83.7), turned to -90 degrees
Routing:
- net +5V: track 32.4 -> 41.1 mm, vias 8 -> 9
- net 3.3V Output: track 50.0 -> 53.7 mm, vias 12 -> 13
- net Net-(U4-NR): track 0.00 -> 1.77 mm
- net GND: track 26.3 -> 27.5 mm, vias 173 -> 174
