File: pcb/Evan_-5V_and_signal_gen.kicad_sch (KiCad schematic)
At the start: 36 parts, among them IC1 TL7660IDGKR, IC2 TL081IDT, U2 LTC4300A-1IMS8_PBF, U4 TPS79933QDDCRQ1, U5 TPS2069CDBVR_MOSFET

Commit message: Updated BOM
Parts:
- C12, C13: MPN (none) -> C0805C106M4RALTU; Manufacturer (none) -> KEMET; Manufacturer_Part_Number T495D106K035ATE300 -> (none)
- C14, C15, C16, C17: MPN (none) -> KGM05AR51A474KH; Manufacturer (none) -> KYOCERA AVX
- C18, C41, C44, C50: MPN (none) -> C0805C104J4RALTU; Manufacturer (none) -> KEMET
- C19, C26, C43: MPN (none) -> C0402C103J4RALTU; Manufacturer (none) -> KEMET
- C25: MPN (none) -> C0603C225K8RACTU; Manufacturer (none) -> KEMET
- C42: MPN (none) -> CL32A157MQVNNNE; Manufacturer (none) -> Samsung Electro-Mechanics; Manufacturer_Part_Number CL32A157MQVNNNE -> (none)
- C47: MPN (none) -> C0805C475J4RACTU; Manufacturer (none) -> KEMET
- I2C_1, J_SIG1, PWR1: now not fitted
- IC1: MPN (none) -> TL7660IDGKR; Manufacturer (none) -> Texas Instruments; Manufacturer_Part_Number TL7660IDGKR -> (none)
- IC2: MPN (none) -> TL081IDT; Manufacturer (none) -> STMicroelectronics; Manufacturer_Part_Number TL081IDT -> (none)
- R10: value 9K -> 10K; MPN (none) -> CRCW040210K0FKTD; Manufacturer (none) -> Vishay Dale
- R11, R12, R3, R4: MPN (none) -> CRCW040210K0FKTD; Manufacturer (none) -> Vishay Dale
- R32: MPN (none) -> CRCW040256K0FKTD; Manufacturer (none) -> Vishay Dale
- R33: MPN (none) -> CRCW0402200RFKTD; Manufacturer (none) -> Vishay Dale
- R5, R6, R7, R8: MPN (none) -> CRCW04023K30FKTD; Manufacturer (none) -> Vishay Dale
- R9: MPN (none) -> CRCW04021K00FKTD; Manufacturer (none) -> Vishay Dale
- U2: MPN (none) -> LTC4300A-1IMS8#PBF; Manufacturer (none) -> Analog Devices Inc.
- U4: MPN (none) -> TPS79933QDDCRQ1; Manufacturer (none) -> Texas Instruments
- U5: MPN (none) -> TPS2069CDBVR; Manufacturer (none) -> Texas Instruments
