File: pcb/mcu_integration.kicad_sch (KiCad schematic)
At the start: 33 parts, among them IC3 LMT87DCKT, J1 Conn_01x05, J5 DM3BT-DSF-PEJS, U1 STM32F103RBTx, Y1 ECS-80-18-5PX-GM-TR

Commit message: Updated BOM
Parts:
- C1, C2, C20, C27, C3, C4, C6, C9: MPN (none) -> C0402C104J4RALTU; Manufacturer (none) -> KEMET
- C10, C11, D1, J1, MH1, MH2, MH3, MH4, SH1, SH2, SH3: now not fitted
- C21: MPN (none) -> C0402C221K8RACTU; Manufacturer (none) -> KEMET
- C23: MPN (none) -> C0402C103J4RALTU; Manufacturer (none) -> KEMET
- C33, C7, C8: MPN (none) -> 0402ZD105KAT2A; Manufacturer (none) -> KYOCERA AVX
- C5: MPN (none) -> C0603C106M9PACTU; Manufacturer (none) -> KEMET
- FB1: MPN (none) -> GZ1608E601TF; Manufacturer (none) -> Shenzhen Sunlord Electronics Co., Ltd.
- IC3: MPN (none) -> LMT87DCKT; Manufacturer (none) -> Texas Instruments; Manufacturer_Part_Number LMT87DCKT -> (none)
- J5: MPN (none) -> DM3BT-DSF-PEJS; Manufacturer (none) -> Hirose Electric Co Ltd
- R1: MPN (none) -> CRCW04022K20FKTD; Manufacturer (none) -> Vishay Dale
- R2: MPN (none) -> CRCW04022K20FKTD; Manufacturer (none) -> Vishay Dale; now not fitted
- S1: MPN (none) -> 95C04A3GWRT; Manufacturer (none) -> Grayhill Inc.; Manufacturer_Part_Number 95C04A3GWRT -> (none)
- U1: MPN (none) -> STM32F103RBT6; Manufacturer (none) -> STMicroelectronics
- Y1: Manufacturer_Part_Number ECS-80-18-5PX-GM-TR -> (none); now not fitted
