File: pcb/untitled.kicad_sch (KiCad schematic)
At the start: 17 parts, among them IC6 AD844_OPAMP_AL, IC7 FOD814_OPTO_AL, J2 Conn_01x03, U3 REF192_AL

Commit message: Updated BOM
Parts:
- C22: MPN (none) -> C0805C106M4RALTU; Manufacturer (none) -> KEMET; Manufacturer_Part_Number T495D106K035ATE300 -> (none)
- C28, C32: MPN (none) -> C0805C104J4RALTU; Manufacturer (none) -> KEMET
- C29, C30: MPN (none) -> C0805C224J4RALTU; Manufacturer (none) -> KEMET; Manufacturer_Part_Number C0805C224M5VACTU -> (none)
- C31: MPN (none) -> C0805C105J4RALTU; Manufacturer (none) -> KEMET; Manufacturer_Part_Number C0805C105Z5VACTU -> (none)
- IC6: MPN (none) -> AD844JRZ-16-REEL7; Manufacturer (none) -> Analog Devices Inc.; Manufacturer_Part_Number AD844JRZ-16-REEL7 -> (none)
- IC7: MPN (none) -> FOD814SD; Manufacturer (none) -> onsemi; Manufacturer_Part_Number FOD814SD -> (none)
- J2, J_AD2: now not fitted
- R22: MPN (none) -> CRCW0402100KFKTD; Manufacturer (none) -> Vishay Dale
- R23: MPN (none) -> CRCW0402820RFKED; Manufacturer (none) -> Vishay Dale
- R24: MPN (none) -> CRCW040247R0FKTD; Manufacturer (none) -> Vishay Dale
- R25: MPN (none) -> CRCW04021K00FKTD; Manufacturer (none) -> Vishay Dale
- R26, R27: MPN (none) -> CRCW0402100RFKTD; Manufacturer (none) -> Vishay Dale
- U3: MPN (none) -> REF192GSZ; Manufacturer (none) -> Analog Devices Inc.
